File: Electronics/MainBoard/MainBoard.kicad_pcb (KiCad board)
At the start: 2 copper layers, 57.8 x 31.1 mm, 30 parts, among them J1 CONN_02X04, J2 DB9_Female, M1 Vibr_Motor, Q1 2N 2222A, Q2 2N 2222A, Q3 2N 2222A, Q4 2N 2222A, Q5 2N 2222A, SW1 SW_PUSH, SW2 SPST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

Commit message: {Began revamp of PCB for professional manufacture!}
Parts:
- removed REF***: OSHW-Logo2_9.8x8mm_Copper, Symbols:OSHW-Logo2_9.8x8mm_Copper
- added C3: 100nF, Resistors_SMD:R_1210, B.Cu at (137.4, 96.6)
- added D3: Flyback, Diodes_SMD:SOD-323_HandSoldering, B.Cu at (154.3, 101.5)
- added P1: BAT_CHG, Pin_Headers:Pin_Header_Straight_1x02, F.Cu at (132.6, 101.2)
- added R2: I2C, Resistors_SMD:R_0603_HandSoldering, B.Cu at (167.6, 100.5)
- added R3: I2C, Resistors_SMD:R_0603_HandSoldering, B.Cu at (166.1, 100.5)
- C1, C2: value C_Small -> 22pF
- D1: footprint LEDs:LED_D3.0mm_Horizontal_O1.27mm_Z10.0mm -> Pin_Headers:Pin_Header_Straight_1x02_Pitch2.00mm
- D2: footprint LEDs:LED_D5.0mm-4 -> Pin_Headers:Pin_Header_Straight_1x04_Pitch2.00mm
- R1: value 470Ω -> 1kΩ
- R6: value 1MΩ -> RST
- RN3: value 220Ω -> 1kΩ
- SW2: footprint Pin_Headers:Pin_Header_Straight_1x03_Pitch2.54mm -> Pin_Headers:Pin_Header_Straight_1x02_Pitch2.00mm
- moved D2 3.24 mm to (116.8, 106.0), turned to 180 degrees
- moved D1 2.25 mm to (116.8, 95.6), turned to 0 degrees
- moved SW2 0.52 mm to (128.8, 106.8)
Routing:
- net Net-(D2-Pad4): track 30.5 -> 0.00 mm
- net Net-(D2-Pad3): track 29.9 -> 0.00 mm
- net Net-(D2-Pad1): track 27.0 -> 0.00 mm, vias 1 -> 0
- net /SDA: track 31.8 -> 39.2 mm
- net Net-(D1-Pad1): track 17.6 -> 14.6 mm
- net GND: track 37.8 -> 40.0 mm, vias 2 -> 3
- net /SCL: track 35.2 -> 37.2 mm
- net +3V3: track 43.2 -> 45.2 mm
- net Net-(D3-Pad2): track 2.93 -> 4.91 mm
- net /TRG: track 27.2 -> 26.5 mm
