File: Electronics/MainBoard/MainBoard.sch (KiCad schematic (older format))
At the start: 29 parts, among them J1 CONN_02X04, J2 DB9_Female, M1 Vibr_Motor, Q1 2N 2222A, Q2 2N 2222A, Q3 2N 2222A, Q4 2N 2222A, Q5 2N 2222A, SW1 SW_PUSH, SW2 SPST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

Commit message: {Began revamp of PCB for professional manufacture!}
Parts:
- added C3: 100nF, Resistors_SMD:R_1210, symbol C_Small
- added D3: Flyback, Diodes_SMD:SOD-323_HandSoldering, symbol D_Small
- added P1: BAT_CHG, Pin_Headers:Pin_Header_Straight_1x02, symbol CONN_01X02
- added R2, R3: I2C, Resistors_SMD:R_0603_HandSoldering, symbol R_Small
- C1, C2: value C_Small -> 22pF
- D1: footprint LEDs:LED_D3.0mm_Horizontal_O1.27mm_Z10.0mm -> Pin_Headers:Pin_Header_Straight_1x02_Pitch2.00mm
- D2: footprint LEDs:LED_D5.0mm-4 -> Pin_Headers:Pin_Header_Straight_1x04_Pitch2.00mm
- R1: value 470Ω -> 1kΩ
- R6: value 1MΩ -> RST
- RN3: value 220Ω -> 1kΩ
- SW2: footprint Pin_Headers:Pin_Header_Straight_1x03_Pitch2.54mm -> Pin_Headers:Pin_Header_Straight_1x02_Pitch2.00mm
Connections:
- net +3V3: now also C3.1, D3.1 (K), R2.1, R3.1
- net GND: now also C3.2, P1.2 (P2)
- net SCL: now also R3.2
- net SDA: now also R2.2
- net at BT1.1, C4.1, SW2.1: now also P1.1 (P1)
- net at M1.1 (GND), Q5.3 (C): now also D3.2 (A)
Changed lines of the file:
@@
 EESchema Schematic File Version 2
-LIBS:MainBoard-rescue
 LIBS:power
 LIBS:device
@@
 P 8400 3000
 F 0 "C1" H 8410 3070 50  0000 L CNN
-F 1 "C_Small" H 8410 2920 50  0000 L CNN
+F 1 "22pF" H 8410 2920 50  0000 L CNN
 F 2 "Capacitors_SMD:C_0603_HandSoldering" H 8400 3000 50  0001 C CNN
 F 3 "" H 8400 3000 50  0000 C CNN
@@
 P 8400 3200
 F 0 "C2" H 8410 3270 50  0000 L CNN
-F 1 "C_Small" H 8410 3120 50  0000 L CNN
+F 1 "22pF" H 8410 3120 50  0000 L CNN
 F 2 "Capacitors_SMD:C_0603_HandSoldering" H 8400 3200 50  0001 C CNN
 F 3 "" H 8400 3200 50  0000 C CNN
@@
 F 0 "D1" H 2400 2675 50  0000 C CNN
 F 1 "LED" H 2400 2475 50  0000 C CNN
-F 2 "LEDs:LED_D3.0mm_Horizontal_O1.27mm_Z10.0mm" H 2400 2575 50  0001 C CNN
+F 2 "Pin_Headers:Pin_Header_Straight_1x02_Pitch2.00mm" H 2400 2575 50  0001 C CNN
 F 3 "" H 2400 2575 50  0000 C CNN
 	1    2400 2575
@@
 F 0 "D2" H 2100 3825 50  0000 C CNN
 F 1 "LED_RCBG" H 2100 3125 50  0000 C CNN
-F 2 "LEDs:LED_D5.0mm-4" H 2100 3425 50  0001 C CNN
+F 2 "Pin_Headers:Pin_Header_Straight_1x04_Pitch2.00mm" H 2100 3425 50  0001 C CNN
 F 3 "" H 2100 3425 50  0000 C CNN
 	1    2100 3475
@@
 P 7950 2150
 F 0 "R6" H 7980 2170 50  0000 L CNN
-F 1 "1MΩ" H 7980 2110 50  0000 L CNN
+F 1 "RST" H 7980 2110 50  0000 L CNN
 F 2 "Resistors_SMD:R_0603_HandSoldering" H 7950 2150 50  0001 C CNN
 F 3 "https://www.reichelt.de/SMD-0603-von-1-bis-910-kOhm/RND-0603-1-100K/3/index.html?ACTION=3&LA=2&ARTICLE=183102&GROUPID=7968&artnr=RND+0603+1+100K&trstct=pol_1;SID=94WOY5-qwQATcAAG79Goo0acb105dd429f907499a137e0497339a" H 7950 2150 50  0001 C CNN
@@
 F 0 "SW2" H 10250 5150 50  0000 C CNN
 F 1 "SPST" H 10250 4950 50  0000 C CNN
-F 2 "Pin_Headers:Pin_Header_Straight_1x03_Pitch2.54mm" H 10250 5050 50  0001 C CNN
+F 2 "Pin_Headers:Pin_Header_Straight_1x02_Pitch2.00mm" H 10250 5050 50  0001 C CNN
 F 3 "" H 10250 5050 50  0000 C CNN
 	1    10250 5050
@@
 P 9300 3250
 F 0 "RN3" V 9000 3250 50  0000 C CNN
-F 1 "220Ω" V 9500 3250 50  0000 C CNN
+F 1 "1kΩ" V 9500 3250 50  0000 C CNN
 F 2 "Resistors_SMD:R_Array_Convex_4x0603" V 9575 3250 50  0001 C CNN
 F 3 "https://www.reichelt.de/4-Widerstaende-SMD-1206/BCN16-220/3/index.html?ACTION=3&LA=2&ARTICLE=42464&GROUPID=4495&artnr=BCN16+220&trstct=pol_0" H 9300 3250 50  0001 C CNN
@@
 	10250 5900 10250 5925
 Wire Wire Line
-	10250 5900 9925 5900
+	9925 5900 10700 5900
 Wire Wire Line
 	10250 5550 10250 5600
 Wire Wire Line
-	10250 5575 9925 5575
+	9925 5575 10700 5575
 Connection ~ 10250 5575
 Wire Wire Line
@@
 P 5025 6850
 F 0 "R1" H 5055 6870 50  0000 L CNN
-F 1 "470Ω" H 5055 6810 50  0000 L CNN
+F 1 "1kΩ" H 5055 6810 50  0000 L CNN
 F 2 "Resistors_SMD:R_0603_HandSoldering" H 5025 6850 50  0001 C CNN
 F 3 "" H 5025 6850 50  0001 C CNN
@@
 Text Label 8050 5700 0    60   ~ 0
 V_VBR
+$Comp
+L C_Small C3
+U 1 1 5B5B6917
+P 4950 2850
+F 0 "C3" H 4960 2920 50  0000 L CNN
+F 1 "100nF" H 4960 2770 50  0000 L CNN
+F 2 "Resistors_SMD:R_1210" H 4950 2850 50  0001 C CNN
+F 3 "https://www.reichelt.de/vielschicht-kerko-100nf-100v-125-c-kem-x7r1210-100n-p207173.html?" H 4950 2850 50  0001 C CNN
+	1    4950 2850
+	1    0    0    -1
+$EndComp
+$Comp
+L GND #PWR022
+U 1 1 5B5B6FEC
+P 4950 3050
+F 0 "#PWR022" H 4950 2800 50  0001 C CNN
+F 1 "GND" H 4950 2900 50  0000 C CNN
+F 2 "" H 4950 3050 50  0000 C CNN
+F 3 "" H 4950 3050 50  0000 C CNN
+	1    4950 3050
+	1    0    0    -1
+$EndComp
+Wire Wire Line
+	4950 3050 4950 2950
+Wire Wire Line
+	4950 2750 4950 2650
+Wire Wire Line
+	4950 2650 5200 2650
+Connection ~ 5200 2650
+$Comp
+L D_Small D3
+U 1 1 5B5BAEE9
+P 5250 6500
+F 0 "D3" H 5200 6580 50  0000 L CNN
+F 1 "Flyback" H 5100 6420 50  0000 L CNN
+F 2 "Diodes_SMD:SOD-323_HandSoldering" V 5250 6500 50  0001 C CNN
+F 3 "" V 5250 6500 50  0000 C CNN
+	1    5250 6500
+	0    1    1    0
+$EndComp
+Wire Wire Line
+	5250 6400 5450 6400
+Wire Wire Line
+	5250 6600 5450 6600
+Connection ~ 5450 6600
+$Comp
+L R_Small R2
+U 1 1 5B5C38B0
+P 8050 3700
+F 0 "R2" V 7900 3625 50  0000 L CNN
+F 1 "I2C" V 7975 3625 50  0000 L CNN
+F 2 "Resistors_SMD:R_0603_HandSoldering" H 8050 3700 50  0001 C CNN
+F 3 "" H 8050 3700 50  0000 C CNN
+	1    8050 3700
+	0    1    1    0
+$EndComp
+$Comp
+L R_Small R3
+U 1 1 5B5C3A9B
+P 8050 3800
+F 0 "R3" V 8125 3725 50  0000 L CNN
+F 1 "I2C" V 8200 3725 50  0000 L CNN
+F 2 "Resistors_SMD:R_0603_HandSoldering" H 8050 3800 50  0001 C CNN
+F 3 "" H 8050 3800 50  0000 C CNN
+	1    8050 3800
+	0    1    1    0
+$EndComp
+Wire Wire Line
+	8150 3700 8150 3800
+Wire Wire Line
+	8150 3700 8200 3700
+Wire Wire Line
+	8200 3700 8200 3650
+$Comp
+L +3.3V #PWR023
+U 1 1 5B5C4F46
+P 8200 3650
+F 0 "#PWR023" H 8200 3500 50  0001 C CNN
+F 1 "+3.3V" H 8200 3790 50  0000 C CNN
+F 2 "" H 8200 3650 50  0000 C CNN
+F 3 "" H 8200 3650 50  0000 C CNN
+	1    8200 3650
+	1    0    0    -1
+$EndComp
+Wire Wire Line
+	7950 3700 7600 3700
+Wire Wire Line
+	7950 3800 7600 3800
+Entry Wire Line
+	7500 3800 7600 3700
+Entry Wire Line
+	7500 3900 7600 3800
+Text Label 7650 3800 0    60   ~ 0
+SCL
+Text Label 7650 3700 0    60   ~ 0
+SDA
+$Comp
+L CONN_01X02 P1
+U 1 1 5B5B9316
+P 10900 5750
+F 0 "P1" H 10900 5900 50  0000 C CNN
+F 1 "BAT_CHG" V 11000 5750 50  0000 C CNN
+F 2 "Pin_Headers:Pin_Header_Straight_1x02" H 10900 5750 50  0001 C CNN
+F 3 "" H 10900 5750 50  0000 C CNN
+	1    10900 5750
+	1    0    0    -1
+$EndComp
+Wire Wire Line
+	10700 5575 10700 5700
+Wire Wire Line
+	10700 5900 10700 5800
+Connection ~ 10250 5900
 $EndSCHEMATC
